Commit message: Moved CANOpen driver to herox_base, fixed some stuff so the simulation will run

File: herox_description/urdf/accessories.urdf.xacro (robot description, xacro)
@@ -9,7 +9,7 @@
     ridgeback_base/launch/base.launch
   -->
-  <xacro:include filename="$(find ridgeback_description)/urdf/accessories/sick_lms1xx_mount.urdf.xacro" />
-  <xacro:include filename="$(find ridgeback_description)/urdf/accessories/sick_s300_mount.urdf.xacro" />
-  <xacro:include filename="$(find ridgeback_description)/urdf/accessories/hokuyo_ust-10lx_mount.urdf.xacro" />
+  <xacro:include filename="$(find herox_description)/urdf/accessories/sick_lms1xx_mount.urdf.xacro" />
+  <xacro:include filename="$(find herox_description)/urdf/accessories/sick_s300_mount.urdf.xacro" />
+  <xacro:include filename="$(find herox_description)/urdf/accessories/hokuyo_ust-10lx_mount.urdf.xacro" />
   <!-- If enabled, generate the front HOKUYO UST-10LX LASER payload. -->
   <xacro:if value="$(optenv RIDGEBACK_FRONT_HOKUYO_LASER 0)">
@@ -51,5 +51,5 @@
   </xacro:if>
   <!-- If enabled, generate the optional Microstrain 3DM-GX2/3 IMU payload. -->
-  <xacro:include filename="$(find ridgeback_description)/urdf/accessories/microstrain_imu.urdf.xacro" />
+  <xacro:include filename="$(find herox_description)/urdf/accessories/microstrain_imu.urdf.xacro" />
   <xacro:if value="$(optenv RIDGEBACK_MICROSTRAIN_IMU 0)">
     <xacro:microstrain_imu prefix="$(optenv RIDGEBACK_MICROSTRAIN_IMU_PREFIX upgraded)"

File: herox_description/urdf/accessories/hokuyo_ust-10lx_mount.urdf.xacro (robot description, xacro)
@@ -19,5 +19,5 @@
         <geometry>
           <!-- Origin of this mesh is the focal point of the LIDAR. -->
-          <mesh filename="package://ridgeback_description/meshes/ust-10lx.stl" />
+          <mesh filename="package://herox_description/meshes/ust-10lx.stl" />
         </geometry>
         <material name="dark_grey" />

File: herox_description/urdf/herox_amr.urdf.xacro (robot description, xacro)
@@ -41,8 +41,8 @@
       <origin xyz="${wheel_x_offset} ${-(wheel_y_offset)} 0" rpy="0 0 0" />
     </xacro:wheel>
-    <xacro:wheel prefix="back" side="left">
+    <xacro:wheel prefix="rear" side="left">
       <origin xyz="${-(wheel_x_offset)} ${wheel_y_offset} 0" rpy="0 0 0" />
     </xacro:wheel>
-    <xacro:wheel prefix="back" side="right">
+    <xacro:wheel prefix="rear" side="right">
       <origin xyz="${-(wheel_x_offset)} ${-(wheel_y_offset)} 0" rpy="0 0 0" />
     </xacro:wheel>

File: herox_description/urdf/ridgeback.urdf.xacro (robot description, xacro)
@@ -26,5 +26,5 @@
         <origin xyz="0 0 0" rpy="${PI/2} 0 0"/>
         <geometry>
-          <mesh filename="package://ridgeback_description/meshes/wheel.stl"/>
+          <mesh filename="package://herox_description/meshes/wheel.stl"/>
         </geometry>
         <material name="black" />
@@ -66,5 +66,5 @@
         <origin xyz="0 0 0" rpy="${PI/2} 0 ${PI/2}" />
         <geometry>
-          <mesh filename="package://ridgeback_description/meshes/rocker.stl"/>
+          <mesh filename="package://herox_description/meshes/rocker.stl"/>
         </geometry>
         <material name="black" />
@@ -109,5 +109,5 @@
       <origin xyz="0 0 0" rpy="0 0 0" />
       <geometry>
-        <mesh filename="package://ridgeback_description/meshes/body.stl"/>
+        <mesh filename="package://herox_description/meshes/body.stl"/>
       </geometry>
       <material name="black" />
@@ -116,5 +116,5 @@
       <origin xyz="0 0 0"/>
       <geometry>
-        <mesh filename="package://ridgeback_description/meshes/body-collision.stl"/>
+        <mesh filename="package://herox_description/meshes/body-collision.stl"/>
       </geometry>
     </collision>
@@ -142,5 +142,5 @@
       <origin xyz="0 0 0" rpy="0 0 ${PI}" />
       <geometry>
-        <mesh filename="package://ridgeback_description/meshes/side-cover.stl"/>
+        <mesh filename="package://herox_description/meshes/side-cover.stl"/>
       </geometry>
       <material name="yellow" />
@@ -151,5 +151,5 @@
       <origin xyz="0 0 0" rpy="0 0 0" />
       <geometry>
-        <mesh filename="package://ridgeback_description/meshes/side-cover.stl"/>
+        <mesh filename="package://herox_description/meshes/side-cover.stl"/>
       </geometry>
       <material name="yellow" />
@@ -165,5 +165,5 @@
       <origin xyz="0 0 0" rpy="0 0 0" />
       <geometry>
-        <mesh filename="package://ridgeback_description/meshes/end-cover.stl" />
+        <mesh filename="package://herox_description/meshes/end-cover.stl" />
       </geometry>
       <material name="black" />
@@ -179,5 +179,5 @@
       <origin xyz="0 0 0" rpy="0 0 ${PI}" />
       <geometry>
-        <mesh filename="package://ridgeback_description/meshes/end-cover.stl" />
+        <mesh filename="package://herox_description/meshes/end-cover.stl" />
       </geometry>
       <material name="black" />
@@ -198,5 +198,5 @@
       <origin xyz="0 0 0" rpy="0 0 0" />
       <geometry>
-        <mesh filename="package://ridgeback_description/meshes/lights.stl" />
+        <mesh filename="package://herox_description/meshes/lights.stl" />
       </geometry>
       <material name="white" />
@@ -207,5 +207,5 @@
       <origin xyz="0 0 0" rpy="0 0 ${PI}" />
       <geometry>
-        <mesh filename="package://ridgeback_description/meshes/lights.stl" />
+        <mesh filename="package://herox_description/meshes/lights.stl" />
       </geometry>
       <material name="red" />
@@ -221,5 +221,5 @@
       <origin xyz="0 0 0" rpy="0 0 0" />
       <geometry>
-        <mesh filename="package://ridgeback_description/meshes/top.stl" />
+        <mesh filename="package://herox_description/meshes/top.stl" />
       </geometry>
       <material name="black" />
@@ -228,5 +228,5 @@
       <origin xyz="0 0 0" rpy="0 0 0" />
       <geometry>
-        <mesh filename="package://ridgeback_description/meshes/top.stl"/>
+        <mesh filename="package://herox_description/meshes/top.stl"/>
       </geometry>
     </collision>
@@ -241,5 +241,5 @@
       <origin xyz="0 0 0" rpy="0 ${PI/2} 0" />
       <geometry>
-        <mesh filename="package://ridgeback_description/meshes/axle.stl" />
+        <mesh filename="package://herox_description/meshes/axle.stl" />
       </geometry>
       <material name="black" />
@@ -265,9 +265,9 @@
   </joint>
   <!-- Bring in simulation data for Gazebo. -->
-  <xacro:include filename="$(find ridgeback_description)/urdf/ridgeback.gazebo" />
+  <xacro:include filename="$(find herox_description)/urdf/ridgeback.gazebo" />
   <!-- Optional standard accessories, including their simulation data. The rendering
        of these into the final description is controlled by optenv variables, which
        default each one to off.-->
-  <xacro:include filename="$(find ridgeback_description)/urdf/accessories.urdf.xacro" />
+  <xacro:include filename="$(find herox_description)/urdf/accessories.urdf.xacro" />
   <!-- Optional custom includes. -->
   <xacro:include filename="$(optenv RIDGEBACK_URDF_EXTRAS empty.urdf)" />

Commit message: - Improved HEROX URDF file - Added SICK nanoScan3 lasers to accessories and URDF configs (using SICK LMS1XX model with custom parameters, for simulation and on-device) - Updated XBOX teleop scale from 0.5 to 1.0

File: herox_description/urdf/accessories.urdf.xacro (robot description, xacro)
@@ -10,4 +10,5 @@
   -->
   <xacro:include filename="$(find herox_description)/urdf/accessories/sick_lms1xx_mount.urdf.xacro" />
+  <xacro:include filename="$(find herox_description)/urdf/accessories/sick_nanoscan3_mount.urdf.xacro" />
   <xacro:include filename="$(find herox_description)/urdf/accessories/sick_s300_mount.urdf.xacro" />
   <xacro:include filename="$(find herox_description)/urdf/accessories/hokuyo_ust-10lx_mount.urdf.xacro" />
@@ -29,4 +30,16 @@
                              topic="front/scan"
                              location="1" />
+  </xacro:if>
+  <!-- If enabled, generate the front SICK nanoScan3 LASER payload. -->
+  <xacro:if value="$(optenv HEROX_FRONT_NANOSCAN_LASER 0)">
+    <xacro:sick_nanoscan3_mount prefix="front"
+                             topic="front/scan"
+                             location="1" />
+  </xacro:if>
+  <!-- If enabled, generate the rear SICK nanoScan3 LASER payload. -->
+  <xacro:if value="$(optenv HEROX_REAR_NANOSCAN_LASER 0)">
+    <xacro:sick_nanoscan3_mount prefix="rear"
+                             topic="rear/scan"
+                             location="-1" />
   </xacro:if>
   <!-- If enabled, generate the rear SICK LMS111 LASER payload. -->

File: herox_description/urdf/herox_amr.urdf.xacro (robot description, xacro)
@@ -6,8 +6,17 @@
     <xacro:property name="wheel_y_offset" value="0.1500" />
     <xacro:property name="wheel_x_offset" value="0.2215" />
+    <!-- Height of laser scanners (center point) above ground (base link) -->
+    <xacro:property name="laser_height" value="0.230" />
+    <!-- Offset of laser scanners (center point) from center of vehicle (base link) -->
     <!-- NOTE: This measurement is rough for now! -->
     <!-- NOTE: Z-offset is not modeled yet! -->
     <!-- NOTE: Assuming symmetrical placement of lasers -->
     <xacro:property name="laser_offset" value="0.270" />
+    <material name="dark_grey"><color rgba="0.2 0.2 0.2 1.0" /></material>
+    <material name="light_grey"><color rgba="0.4 0.4 0.4 1.0" /></material>
+    <material name="red"><color rgba="0.8 0.0 0.0 1.0" /></material>
+    <material name="white"><color rgba="0.9 0.9 0.9 1.0" /></material>
+    <material name="yellow"><color rgba="0.8 0.8 0.0 1.0" /></material>
+    <material name="black"><color rgba="0.15 0.15 0.15 1.0" /></material>
     <xacro:macro name="wheel" params="prefix side *joint_pose">
         <link name="${prefix}_${side}_wheel_link">
@@ -19,12 +28,18 @@
           </collision>
             <visual>
-                <origin xyz="0 0 0" rpy="0 0 0"/>
+                <origin xyz="0 0 0" rpy="${PI/2} 0 0"/>
                 <geometry>
                     <cylinder radius="${wheel_radius}" length="${wheel_width}"/>
                 </geometry>
-                <material name="grey">
-                    <color rgba="0.5 0.5 0.5 1.0" />
-                </material>
+                <material name="dark_grey"/>
             </visual>
+          <inertial>
+            <origin xyz="0 0 0" rpy="0 0 0"/>
+            <mass value="5.0"/>
+            <inertia
+              ixx="3.3212e-3" ixy="0" ixz="0"
+              iyy="6.6424e-3" iyz="0"
+              izz="3.3212e-3"/>
+          </inertial>
         </link>
         <joint name="${prefix}_${side}_wheel" type="continuous">
@@ -46,5 +61,61 @@
         </transmission>
     </xacro:macro>
-    <link name="base_link" />
+    <link name="base_link"/>
+    <link name="chassis_top_link">
+        <collision>
+            <origin xyz="0 0 0" rpy="0 0 0"/>
+            <geometry>
+                <box size="0.630 0.435 0.130" />
+            </geometry>
+        </collision>
+        <visual>
+            <origin xyz="0 0 0" rpy="0 0 0"/>
+            <geometry>
+                <box size="0.630 0.435 0.130" />
+            </geometry>
+            <material name="light_grey" />
+        </visual>
+        <inertial>
+            <origin xyz="0 0 0" rpy="0 0 0"/>
+            <mass value="10.0"/>
+            <inertia
+                ixx="4.4744" ixy="0.03098" ixz="0.003647"
+                iyy="7.1624" iyz="0.1228"
+                izz="4.6155"/>
+        </inertial>
+    </link>
+    <link name="chassis_bottom_link">
+        <collision>
+            <origin xyz="0 0 0" rpy="0 0 0"/>
+            <geometry>
+                <box size="0.230 0.435 0.205" />
+            </geometry>
+        </collision>
+        <visual>
+            <origin xyz="0 0 0" rpy="0 0 0"/>
+            <geometry>
+                <box size="0.230 0.435 0.205" />
+            </geometry>
+            <material name="light_grey" />
+        </visual>
+        <inertial>
+            <origin xyz="0 0 0" rpy="0 0 0"/>
+            <mass value="20.0"/>
+            <inertia
+                ixx="4.4744" ixy="0.03098" ixz="0.003647"
+                iyy="7.1624" iyz="0.1228"
+                izz="4.6155"/>
+        </inertial>
+    </link>
+    <joint name="chassis_top_link_joint" type="fixed">
+        <origin xyz="0 0 0.280" rpy="0 0 0"/>
+        <parent link="base_link"/>
+        <child link="chassis_top_link"/>
+    </joint>
+    <joint name="chassis_bottom_link_joint" type="fixed">
+        <origin xyz="0 0 0.1125" rpy="0 0 0"/>
+        <parent link="base_link"/>
+        <child link="chassis_bottom_link"/>
+    </joint>
     <xacro:macro name="laser" params="prefix *joint_pose">
         <link name="${prefix}_laser">
@@ -60,8 +131,14 @@
                     <box size="0.1006 0.1025 0.0802" />
                 </geometry>
-                <material name="yellow">
-                    <color rgba="1.0 1.0 0 1.0" />
-                </material>
+                <material name="yellow" />
             </visual>
+          <inertial>
+            <origin xyz="0 0 0" rpy="0 0 0"/>
+            <mass value="1.5"/>
+            <inertia
+              ixx="3.3212e-3" ixy="0" ixz="0"
+              iyy="6.6424e-3" iyz="0"
+              izz="3.3212e-3"/>
+          </inertial>
         </link>
         <joint name="${prefix}_laser_joint" type="fixed">
@@ -73,21 +150,25 @@
     <!-- Wheels -->
     <xacro:wheel prefix="front" side="left">
-      <origin xyz="${wheel_x_offset} ${wheel_y_offset} 0" rpy="0 0 0" />
+        <origin xyz="${wheel_x_offset} ${wheel_y_offset} ${wheel_radius}" rpy="0 0 0" />
     </xacro:wheel>
     <xacro:wheel prefix="front" side="right">
-      <origin xyz="${wheel_x_offset} ${-(wheel_y_offset)} 0" rpy="0 0 0" />
+        <origin xyz="${wheel_x_offset} ${-(wheel_y_offset)} ${wheel_radius}" rpy="0 0 0" />
     </xacro:wheel>
     <xacro:wheel prefix="rear" side="left">
-      <origin xyz="${-(wheel_x_offset)} ${wheel_y_offset} 0" rpy="0 0 0" />
+        <origin xyz="${-(wheel_x_offset)} ${wheel_y_offset} ${wheel_radius}" rpy="0 0 0" />
     </xacro:wheel>
     <xacro:wheel prefix="rear" side="right">
-      <origin xyz="${-(wheel_x_offset)} ${-(wheel_y_offset)} 0" rpy="0 0 0" />
+        <origin xyz="${-(wheel_x_offset)} ${-(wheel_y_offset)} ${wheel_radius}" rpy="0 0 0" />
     </xacro:wheel>
     <!-- Lasers -->
-    <xacro:laser prefix="front">
-	    <origin xyz="${laser_offset} 0 0" rpy="${PI} 0 0" />
+    <!--<xacro:laser prefix="front">
+        <origin xyz="${laser_offset} 0 ${laser_height}" rpy="${PI} 0 0" />
     </xacro:laser>
     <xacro:laser prefix="rear">
-	    <origin xyz="${-(laser_offset)} 0 0" rpy="${PI} 0 ${PI}" />
-    </xacro:laser>
+        <origin xyz="${-(laser_offset)} 0 ${laser_height}" rpy="${PI} 0 ${PI}" />
+    </xacro:laser>-->
+    <!-- Bring in simulation data for Gazebo -->
+    <xacro:include filename="$(find herox_description)/urdf/herox.gazebo" />
+    <!-- Accessories -->
+    <xacro:include filename="$(find herox_description)/urdf/accessories.urdf.xacro" />
 </robot>

Commit message: Removed unnecessary accessory configuration logic from herox_amr URDF as this is robot only comes in one configuration (for now) and this makes things easier

File: herox_description/urdf/accessories.urdf.xacro (robot description, xacro)
@@ -10,5 +10,4 @@
   -->
   <xacro:include filename="$(find herox_description)/urdf/accessories/sick_lms1xx_mount.urdf.xacro" />
-  <xacro:include filename="$(find herox_description)/urdf/accessories/sick_nanoscan3_mount.urdf.xacro" />
   <xacro:include filename="$(find herox_description)/urdf/accessories/sick_s300_mount.urdf.xacro" />
   <xacro:include filename="$(find herox_description)/urdf/accessories/hokuyo_ust-10lx_mount.urdf.xacro" />
@@ -30,16 +29,4 @@
                              topic="front/scan"
                              location="1" />
-  </xacro:if>
-  <!-- If enabled, generate the front SICK nanoScan3 LASER payload. -->
-  <xacro:if value="$(optenv HEROX_FRONT_NANOSCAN_LASER 0)">
-    <xacro:sick_nanoscan3_mount prefix="front"
-                             topic="front/scan"
-                             location="1" />
-  </xacro:if>
-  <!-- If enabled, generate the rear SICK nanoScan3 LASER payload. -->
-  <xacro:if value="$(optenv HEROX_REAR_NANOSCAN_LASER 0)">
-    <xacro:sick_nanoscan3_mount prefix="rear"
-                             topic="rear/scan"
-                             location="-1" />
   </xacro:if>
   <!-- If enabled, generate the rear SICK LMS111 LASER payload. -->

File: herox_description/urdf/accessories/sick_nanoscan3_mount.urdf.xacro (robot description, xacro)
@@ -28,9 +28,15 @@
   <xacro:include filename="$(find lms1xx)/urdf/sick_lms1xx.urdf.xacro" />
   <xacro:macro name="sick_nanoscan3_mount" params="prefix topic location">
+    <!-- Height of laser scanners (center point) above ground (base link) -->
+    <xacro:property name="laser_height" value="0.200" />
+    <!-- Offset of laser scanners (center point) from center of vehicle (base link) -->
+    <!-- NOTE: This measurement is rough for now! -->
+    <!-- NOTE: Z-offset is not modeled yet! -->
+    <!-- NOTE: Assuming symmetrical placement of lasers -->
+    <xacro:property name="laser_offset" value="0.270" />
     <xacro:sick_lms1xx frame="${prefix}_laser" topic="${topic}" max_range="10.0" min_angle="-2.3998" max_angle="2.3998" update_rate="33.0"/>
     <joint name="${prefix}_laser_joint" type="fixed">
         <!-- This offset is from the base_link to the laser scanner's focal point -->
-        <!-- <origin xyz="${location * 0.270} 0 0.230" rpy="0 0 ${PI/2 - (location * PI/2)}" /> -->
-        <origin xyz="${location * 0.270} 0 0.200" rpy="${PI} 0 ${PI/2 - (location * PI/2)}" />
+	<origin xyz="${location * laser_offset} 0 ${laser_height}" rpy="${PI} 0 ${PI/2 - (location * PI/2)}" />
       <parent link="base_link" />
       <child link="${prefix}_laser" />

File: herox_description/urdf/herox_amr.urdf.xacro (robot description, xacro)
@@ -6,11 +6,5 @@
     <xacro:property name="wheel_y_offset" value="0.1500" />
     <xacro:property name="wheel_x_offset" value="0.2215" />
-    <!-- Height of laser scanners (center point) above ground (base link) -->
-    <xacro:property name="laser_height" value="0.230" />
-    <!-- Offset of laser scanners (center point) from center of vehicle (base link) -->
-    <!-- NOTE: This measurement is rough for now! -->
-    <!-- NOTE: Z-offset is not modeled yet! -->
-    <!-- NOTE: Assuming symmetrical placement of lasers -->
-    <xacro:property name="laser_offset" value="0.270" />
+    <xacro:include filename="$(find herox_description)/urdf/accessories/sick_nanoscan3_mount.urdf.xacro" />
     <material name="dark_grey"><color rgba="0.2 0.2 0.2 1.0" /></material>
     <material name="light_grey"><color rgba="0.4 0.4 0.4 1.0" /></material>
@@ -118,34 +112,4 @@
         <child link="chassis_bottom_link"/>
     </joint>
-    <xacro:macro name="laser" params="prefix *joint_pose">
-        <link name="${prefix}_laser">
-            <collision>
-                <origin xyz="0 0 0" rpy="0 0 0"/>
-                <geometry>
-                    <box size="0.1006 0.1025 0.0802" />
-                </geometry>
-            </collision>
-            <visual>
-                <origin xyz="0 0 0" rpy="0 0 0"/>
-                <geometry>
-                    <box size="0.1006 0.1025 0.0802" />
-                </geometry>
-                <material name="yellow" />
-            </visual>
-          <inertial>
-            <origin xyz="0 0 0" rpy="0 0 0"/>
-            <mass value="1.5"/>
-            <inertia
-              ixx="3.3212e-3" ixy="0" ixz="0"
-              iyy="6.6424e-3" iyz="0"
-              izz="3.3212e-3"/>
-          </inertial>
-        </link>
-        <joint name="${prefix}_laser_joint" type="fixed">
-            <parent link="base_link"/>
-            <child link="${prefix}_laser"/>
-            <xacro:insert_block name="joint_pose"/>
-        </joint>
-    </xacro:macro>
     <!-- Wheels -->
     <xacro:wheel prefix="front" side="left">
@@ -162,13 +126,11 @@
     </xacro:wheel>
     <!-- Lasers -->
-    <!--<xacro:laser prefix="front">
-        <origin xyz="${laser_offset} 0 ${laser_height}" rpy="${PI} 0 0" />
-    </xacro:laser>
-    <xacro:laser prefix="rear">
-        <origin xyz="${-(laser_offset)} 0 ${laser_height}" rpy="${PI} 0 ${PI}" />
-    </xacro:laser>-->
+    <xacro:sick_nanoscan3_mount prefix="front"
+                 topic="front/scan"
+                 location="1" />
+    <xacro:sick_nanoscan3_mount prefix="rear"
+                 topic="rear/scan"
+                 location="-1" />
     <!-- Bring in simulation data for Gazebo -->
     <xacro:include filename="$(find herox_description)/urdf/herox.gazebo" />
-    <!-- Accessories -->
-    <xacro:include filename="$(find herox_description)/urdf/accessories.urdf.xacro" />
 </robot>
